Commit message: Updates to the Self tuning regulator

File: src/rover_control/description/gazebo.xacro (robot description, xacro)
@@ -30,5 +30,5 @@
       <joint_name>pendulum_joint</joint_name>
       <topic>joint_states</topic>
-      <update_rate>50</update_rate>
+      <update_rate>100</update_rate>
     </plugin>
   </gazebo>

File: src/rover_control/description/pendulum.urdf.xacro (robot description, xacro)
@@ -20,6 +20,6 @@
     <inertial>
       <origin xyz="0 0 0" rpy="0 0 0"/>
-      <mass value="1000.0"/>
-      <inertia ixx="84.1666667" iyy="84.1666667" izz="166.6666667"
+      <mass value="100.0"/>
+      <inertia ixx="8.416667" iyy="8.416667" izz="16.66667"
                ixy="0" ixz="0" iyz="0"/>
     </inertial>
@@ -52,5 +52,5 @@
       <origin xyz="0 0 0.5" rpy="0 0 0"/>
       <mass value="6.7"/>
-      <inertia ixx="2.23333" iyy="2.23333" izz="0.57229167"
+      <inertia ixx="2.2333" iyy="2.2333" izz="0.0014"
                ixy="0" ixz="0" iyz="0"/>
     </inertial>

Commit message: self_tuning_regulator: Able to stabilize at angle = 0.0

File: src/rover_control/description/gazebo.xacro (robot description, xacro)
@@ -1,5 +1,5 @@
 <?xml version="1.0"?>
 <robot xmlns:xacro="http://www.ros.org/wiki/xacro">
-  <gazebo reference="base_link">
+ <gazebo reference="base_link">
     <mu1>1.0</mu1>
     <mu2>1.0</mu2>
@@ -9,6 +9,6 @@
   </gazebo>
   <gazebo reference="pendulum_link">
-    <mu1>0.2</mu1>
-    <mu2>0.2</mu2>
+    <mu1>1.0</mu1>
+    <mu2>1.0</mu2>
     <kp>1000000.0</kp>
     <kd>100.0</kd>
@@ -19,9 +19,9 @@
         <implicit_spring_damper>true</implicit_spring_damper>
         <cfm_damping>true</cfm_damping>
-        <cfm>0.000001</cfm>
+        <cfm>0.00001</cfm>
         <erp>0.2</erp>
       </ode>
     </physics>
-    <dynamics damping="0.02" friction="0.01"/>
+    <dynamics damping="0.5" friction="0.5"/>
   </gazebo>
   <gazebo>
@@ -30,5 +30,5 @@
       <joint_name>pendulum_joint</joint_name>
       <topic>joint_states</topic>
-      <update_rate>20</update_rate>
+      <update_rate>1000</update_rate>
     </plugin>
   </gazebo>

File: src/rover_control/description/pendulum_free.urdf.xacro (robot description, xacro)
@@ -56,5 +56,5 @@
   <joint name="pendulum_joint" type="continuous">
     <!-- <limit effort="30.0" lower="-3.1415" upper="3.1415" velocity="30.0"/> -->
-    <limit effort="10.0" velocity="10.0"/>
+    <limit effort="50.0" velocity="30.0"/>
     <parent link="column_link"/>
     <child link="pendulum_link"/>
@@ -82,5 +82,5 @@
       <origin xyz="0 0 0.25" rpy="0 0 0"/>
       <mass value="0.135"/>
-      <inertia ixx="0.003" iyy="0.003" izz="0.0"
+      <inertia ixx="0.01125" iyy="0.01125" izz="0.0001"
                ixy="0.0" ixz="0.0" iyz="0.0"/>
     </inertial>

Commit message: self_tuning_regulator: changes to simulation structure

File: src/rover_control/description/gazebo.xacro (robot description, xacro)
@@ -8,21 +8,28 @@
     <kd>100.0</kd>
   </gazebo>
-  <gazebo reference="pendulum_link">
+ <gazebo reference="column_link">
     <mu1>1.0</mu1>
     <mu2>1.0</mu2>
+    <static>true</static>
     <kp>1000000.0</kp>
     <kd>100.0</kd>
   </gazebo>
-  <gazebo reference="pendulum_joint">
-    <physics>
-      <ode>
-        <implicit_spring_damper>true</implicit_spring_damper>
-        <cfm_damping>true</cfm_damping>
-        <cfm>0.00001</cfm>
-        <erp>0.2</erp>
-      </ode>
-    </physics>
-    <dynamics damping="0.5" friction="0.5"/>
+  <gazebo reference="pendulum_link">
+    <mu1>0.5</mu1>
+    <mu2>0.5</mu2>
+    <kp>1000000.0</kp>
+    <kd>100.0</kd>
   </gazebo>
+  <!-- <gazebo reference="pendulum_joint"> -->
+  <!--   <physics> -->
+  <!--     <ode> -->
+  <!--       <implicit_spring_damper>true</implicit_spring_damper> -->
+  <!--       <cfm_damping>true</cfm_damping> -->
+  <!--       <cfm>0.00001</cfm> -->
+  <!--       <erp>0.5</erp> -->
+  <!--     </ode> -->
+  <!--   </physics> -->
+  <!--   <dynamics damping="10.0" friction="5.0"/> -->
+  <!-- </gazebo> -->
   <gazebo>
     <plugin filename="gz-sim-joint-state-publisher-system"
@@ -30,5 +37,5 @@
       <joint_name>pendulum_joint</joint_name>
       <topic>joint_states</topic>
-      <update_rate>1000</update_rate>
+      <update_rate>100</update_rate>
     </plugin>
   </gazebo>

File: src/rover_control/description/pendulum_free.urdf.xacro (robot description, xacro)
@@ -1,5 +1,5 @@
 <?xml version="1.0"?>
 <robot xmlns:xacro="http://www.ros.org/wiki/xacro" name="pendulum">
-  <xacro:include filename="$(find rover_control)/description/gazebo.xacro"/>
+  <!-- <xacro:include filename="$(find rover_control)/description/gazebo.xacro"/> -->
   <link name="base_link">
     <visual>
@@ -54,15 +54,16 @@
     </inertial>
   </link>
+  <!-- <limit effort="30.0" lower="-3.1415" upper="3.1415" velocity="30.0"/> -->
   <joint name="pendulum_joint" type="continuous">
-    <!-- <limit effort="30.0" lower="-3.1415" upper="3.1415" velocity="30.0"/> -->
-    <limit effort="50.0" velocity="30.0"/>
+    <limit effort="100.0" velocity="100.0"/>
     <parent link="column_link"/>
     <child link="pendulum_link"/>
-    <origin xyz="-0.1005 0.0 0.5" rpy="0 0 0"/>
-    <axis xyz="1 0 0"/>
+    <origin xyz="-0.107 0.0 0.5" rpy="0 0 0"/>
+    <axis xyz="-1 0 0"/>
+    <dynamics damping="1.0" friction="0.5"/>
   </joint>
   <link name="pendulum_link">
     <visual>
-      <origin xyz="0 0 0.25" rpy="0 0 0"/>
+      <origin xyz="0 0 -0.25" rpy="0 0 0"/>
       <geometry>
         <box size="0.01 0.01 0.5"/>
@@ -73,5 +74,5 @@
     </visual>
     <collision>
-      <origin xyz="0 0 0.25" rpy="0 0 0"/>
+      <origin xyz="0 0 -0.25" rpy="0 0 0"/>
       <geometry>
         <box size="0.01 0.01 0.5"/>
@@ -79,8 +80,7 @@
     </collision>
     <inertial>
-<!-- Using an aluminium bar as the pendulum link \rho=2.7 g/cm^3-->
-      <origin xyz="0 0 0.25" rpy="0 0 0"/>
-      <mass value="0.135"/>
-      <inertia ixx="0.01125" iyy="0.01125" izz="0.0001"
+      <origin xyz="0 0 -0.25" rpy="0 0 0"/>
+      <mass value="0.5"/>
+      <inertia ixx="0.04167" iyy="0.04167" izz="0.0001"
                ixy="0.0" ixz="0.0" iyz="0.0"/>
     </inertial>
@@ -97,3 +97,17 @@
     </joint>
   </ros2_control>
+  <gazebo>
+    <plugin filename="gz-sim-joint-state-publisher-system"
+            name="gz::sim::systems::JointStatePublisher">
+      <joint_name>pendulum_joint</joint_name>
+      <topic>joint_states</topic>
+      <update_rate>100</update_rate>
+    </plugin>
+  </gazebo>
+  <gazebo>
+    <plugin filename="gz_ros2_control-system"
+            name="gz_ros2_control::GazeboSimROS2ControlPlugin">
+      <parameters>$(find rover_control)/config/pendulum_controller.yaml</parameters>
+    </plugin>
+  </gazebo>
 </robot>
