Commit message: Self Tuning Regulator Fixes

File: src/rover_control/description/pendulum_free.urdf.xacro (robot description, xacro)
@@ -64,7 +64,7 @@
   <link name="pendulum_link">
     <visual>
-      <origin xyz="0 0 0.5" rpy="0 0 0"/>
+      <origin xyz="0 0 0.25" rpy="0 0 0"/>
       <geometry>
-        <box size="0.05 0.05 1.0"/>
+        <box size="0.01 0.01 0.5"/>
       </geometry>
       <material name="pendulum_color">
@@ -73,14 +73,14 @@
     </visual>
     <collision>
-      <origin xyz="0 0 0.5" rpy="0 0 0"/>
+      <origin xyz="0 0 0.25" rpy="0 0 0"/>
       <geometry>
-        <box size="0.05 0.05 1.0"/>
+        <box size="0.01 0.01 0.5"/>
       </geometry>
     </collision>
     <inertial>
 <!-- Using an aluminium bar as the pendulum link \rho=2.7 g/cm^3-->
-      <origin xyz="0 0 0.5" rpy="0 0 0"/>
-      <mass value="6.7"/>
-      <inertia ixx="2.2333" iyy="2.2333" izz="0.0014"
+      <origin xyz="0 0 0.25" rpy="0 0 0"/>
+      <mass value="0.135"/>
+      <inertia ixx="0.003" iyy="0" izz="0.003"
                ixy="0" ixz="0" iyz="0"/>
     </inertial>

Commit message: Self Tuning Regulator update

File: src/rover_control/description/pendulum_free.urdf.xacro (robot description, xacro)
@@ -56,8 +56,8 @@
   <joint name="pendulum_joint" type="continuous">
     <!-- <limit effort="30.0" lower="-3.1415" upper="3.1415" velocity="30.0"/> -->
-    <limit effort="30.0" velocity="30.0"/>
+    <limit effort="10.0" velocity="10.0"/>
     <parent link="column_link"/>
     <child link="pendulum_link"/>
-    <origin xyz="-0.125 0.0 0.5" rpy="0 0 0"/>
+    <origin xyz="-0.1005 0.0 0.5" rpy="0 0 0"/>
     <axis xyz="1 0 0"/>
   </joint>
@@ -82,6 +82,6 @@
       <origin xyz="0 0 0.25" rpy="0 0 0"/>
       <mass value="0.135"/>
-      <inertia ixx="0.003" iyy="0" izz="0.003"
-               ixy="0" ixz="0" iyz="0"/>
+      <inertia ixx="0.003" iyy="0.003" izz="0.0"
+               ixy="0.0" ixz="0.0" iyz="0.0"/>
     </inertial>
   </link>

Commit message: self_tuning_regulator: dynamic target angle setting working

File: src/rover_control/description/pendulum_free.urdf.xacro (robot description, xacro)
@@ -56,10 +56,10 @@
   <!-- <limit effort="30.0" lower="-3.1415" upper="3.1415" velocity="30.0"/> -->
   <joint name="pendulum_joint" type="continuous">
-    <limit effort="100.0" velocity="100.0"/>
+    <!-- <limit effort="5.0" velocity="5.0"/> -->
     <parent link="column_link"/>
     <child link="pendulum_link"/>
     <origin xyz="-0.107 0.0 0.5" rpy="0 0 0"/>
     <axis xyz="-1 0 0"/>
-    <dynamics damping="1.0" friction="0.5"/>
+    <dynamics damping="0.30" friction="0.01"/>
   </joint>
   <link name="pendulum_link">
@@ -102,5 +102,5 @@
       <joint_name>pendulum_joint</joint_name>
       <topic>joint_states</topic>
-      <update_rate>100</update_rate>
+      <update_rate>1000</update_rate>
     </plugin>
   </gazebo>
