Commit message: self tuning regulator

File: src/rover_control/description/pendulum.urdf.xacro (robot description, xacro)
@@ -26,5 +26,5 @@
   </link>
   <joint name="pendulum_joint" type="revolute">
-    <limit effort="1000.0" lower="-1.4" upper="1.4" velocity="0.5"/>
+    <limit effort="100.0" lower="-1.3" upper="1.3" velocity="5.0"/>
     <parent link="base_link"/>
     <child link="pendulum_link"/>

Commit message: fixed covariance publisher

File: src/rover_control/description/pendulum.urdf.xacro (robot description, xacro)
@@ -20,11 +20,11 @@
     <inertial>
       <origin xyz="0 0 0" rpy="0 0 0"/>
-      <mass value="10.0"/>
-      <inertia ixx="0.841666667" iyy="0.841666667" izz="1.666666667"
+      <mass value="100.0"/>
+      <inertia ixx="8.41666667" iyy="8.41666667" izz="16.66666667"
                ixy="0" ixz="0" iyz="0"/>
     </inertial>
   </link>
   <joint name="pendulum_joint" type="revolute">
-    <limit effort="100.0" lower="-1.3" upper="1.3" velocity="5.0"/>
+    <limit effort="100.0" lower="-1.3" upper="1.3" velocity="500.0"/>
     <parent link="base_link"/>
     <child link="pendulum_link"/>

Commit message: editted the loggers

File: src/rover_control/description/pendulum.urdf.xacro (robot description, xacro)
@@ -26,5 +26,5 @@
   </link>
   <joint name="pendulum_joint" type="revolute">
-    <limit effort="100.0" lower="-1.3" upper="1.3" velocity="500.0"/>
+    <limit effort="500.0" lower="-1.3" upper="1.3" velocity="500.0"/>
     <parent link="base_link"/>
     <child link="pendulum_link"/>

Commit message: Updated at the Monday 8/4/2025 meeting

File: src/rover_control/description/pendulum.urdf.xacro (robot description, xacro)
@@ -49,7 +49,8 @@
     </collision>
     <inertial>
+<!-- Using an aluminium bar as the pendulum link \rho=2.7 g/cm^3-->
       <origin xyz="0 0 0.5" rpy="0 0 0"/>
-      <mass value="0.5"/>
-      <inertia ixx="0.958333333" iyy="0.958333333" izz="0.000208333"
+      <mass value="6.7"/>
+      <inertia ixx="2.23333" iyy="2.23333" izz="0.57229167"
                ixy="0" ixz="0" iyz="0"/>
     </inertial>

Commit message: Inverted Pendulum is working

File: src/rover_control/description/pendulum.urdf.xacro (robot description, xacro)
@@ -20,6 +20,6 @@
     <inertial>
       <origin xyz="0 0 0" rpy="0 0 0"/>
-      <mass value="100.0"/>
-      <inertia ixx="8.41666667" iyy="8.41666667" izz="16.66666667"
+      <mass value="1000.0"/>
+      <inertia ixx="84.1666667" iyy="84.1666667" izz="166.6666667"
                ixy="0" ixz="0" iyz="0"/>
     </inertial>

Commit message: Adding support for 2 link pendulum

File: src/rover_control/description/pendulum.urdf.xacro (robot description, xacro)
@@ -1,5 +1,4 @@
 <?xml version="1.0"?>
 <robot xmlns:xacro="http://www.ros.org/wiki/xacro" name="pendulum">
-  <xacro:include filename="$(find rover_control)/description/gazebo.xacro"/>
   <link name="base_link">
     <visual>
@@ -20,21 +19,51 @@
     <inertial>
       <origin xyz="0 0 0" rpy="0 0 0"/>
-      <mass value="100.0"/>
+      <mass value="1000.0"/>
       <inertia ixx="8.416667" iyy="8.416667" izz="16.66667"
                ixy="0" ixz="0" iyz="0"/>
     </inertial>
   </link>
-  <joint name="pendulum_joint" type="revolute">
-    <limit effort="500.0" lower="-1.3" upper="1.3" velocity="500.0"/>
+  <joint name="column_joint" type="fixed">
     <parent link="base_link"/>
-    <child link="pendulum_link"/>
-    <origin xyz="0.0 0.0 0.1" rpy="0 0 0"/>
-    <axis xyz="1 0 0"/>
+    <child link="column_link"/>
+    <origin xyz="0.0 0.0 0.75" rpy="0 0 0"/>
+    <axis xyz="0 1 0"/>
   </joint>
-  <link name="pendulum_link">
+  <link name="column_link">
     <visual>
-      <origin xyz="0 0 0.5" rpy="0 0 0"/>
+      <origin xyz="0 0 0.0" rpy="0 0 0"/>
       <geometry>
-        <box size="0.05 0.05 1.0"/>
+        <box size="0.2 0.2 1.5"/>
+      </geometry>
+      <material name="blue">
+        <color rgba="0.2 0.2 0.8 1.0"/>
+      </material>
+    </visual>
+    <collision>
+      <origin xyz="0 0 0" rpy="0 0 0"/>
+      <geometry>
+        <box size="0.2 0.2 1.5"/>
+      </geometry>
+    </collision>
+    <inertial>
+      <origin xyz="0 0 0" rpy="0 0 0"/>
+      <mass value="1000.0"/>
+      <inertia ixx="8.416667" iyy="8.416667" izz="16.66667"
+               ixy="0" ixz="0" iyz="0"/>
+    </inertial>
+  </link>
+  <joint name="pendulum_joint1" type="continuous">
+    <!-- <limit effort="5.0" velocity="5.0"/> -->
+    <parent link="column_link"/>
+    <child link="pendulum_link1"/>
+    <origin xyz="-0.107 0.0 0.5" rpy="0 0 0"/>
+    <axis xyz="-1 0 0"/>
+    <dynamics damping="0.40" friction="0.01"/>
+  </joint>
+  <link name="pendulum_link1">
+    <visual>
+      <origin xyz="0 0 -0.25" rpy="0 0 0"/>
+      <geometry>
+        <box size="0.01 0.01 0.5"/>
       </geometry>
       <material name="pendulum_color">
@@ -43,15 +72,14 @@
     </visual>
     <collision>
-      <origin xyz="0 0 0.5" rpy="0 0 0"/>
+      <origin xyz="0 0 -0.25" rpy="0 0 0"/>
       <geometry>
-        <box size="0.05 0.05 1.0"/>
+        <box size="0.01 0.01 0.5"/>
       </geometry>
     </collision>
     <inertial>
-<!-- Using an aluminium bar as the pendulum link \rho=2.7 g/cm^3-->
-      <origin xyz="0 0 0.5" rpy="0 0 0"/>
-      <mass value="6.7"/>
-      <inertia ixx="2.2333" iyy="2.2333" izz="0.0014"
-               ixy="0" ixz="0" iyz="0"/>
+      <origin xyz="0 0 -0.25" rpy="0 0 0"/>
+      <mass value="0.5"/>
+      <inertia ixx="0.04167" iyy="0.04167" izz="0.0001"
+               ixy="0.0" ixz="0.0" iyz="0.0"/>
     </inertial>
   </link>
@@ -60,9 +88,27 @@
       <plugin>gz_ros2_control/GazeboSimSystem</plugin>
     </hardware>
-    <joint name="pendulum_joint">
+    <joint name="pendulum_joint1">
       <command_interface name="effort"/>
       <state_interface name="position"/>
       <state_interface name="velocity"/>
+      <state_interface name="effort"/>
     </joint>
   </ros2_control>
+  <gazebo>
+    <plugin filename="gz-sim-joint-state-publisher-system"
+            name="gz::sim::systems::JointStatePublisher">
+      <joint_name>pendulum_joint1</joint_name>
+      <topic>joint_states</topic>
+      <update_rate>1000</update_rate>
+    </plugin>
+  </gazebo>
+  <gazebo>
+    <plugin filename="gz_ros2_control-system"
+            name="gz_ros2_control::GazeboSimROS2ControlPlugin">
+      <parameters>$(find rover_control)/config/pendulum_controller.yaml</parameters>
+      <ros>
+        <parameter name="use_sim_time" type="bool">true</parameter>
+      </ros>
+    </plugin>
+  </gazebo>
 </robot>
