Commit message: Fixed build dependencies and errors

File: src/pendulum_control/description/two_link.urdf.xacro (robot description, xacro)
@@ -54,5 +54,5 @@
   </link>
   <joint name="pendulum_joint1" type="continuous">
-    <limit effort="10.0" velocity="5.0"/>
+    <limit effort="10.0" velocity="10.0"/>
     <parent link="column_link"/>
     <child link="pendulum_link1"/>
@@ -85,11 +85,10 @@
   </link>
   <joint name="pendulum_joint2" type="revolute">
-    <!-- <limit effort="5.0" velocity="5.0"/> -->
-    <limit effort="10" velocity="5.0" lower="-3.14159" upper="3.14159" />
+    <limit effort="5.0" velocity="5.0" lower="0.0" upper="6.283" />
     <parent link="pendulum_link1"/>
     <child link="pendulum_link2"/>
     <origin xyz="0.0 0.0 -0.50" rpy="0 0 0"/>
     <axis xyz="-1 0 0"/>
-    <dynamics damping="0.50" friction="0.03"/>
+    <dynamics damping="0.50" friction="0.01"/>
   </joint>
   <link name="pendulum_link2">
